Commit message: Add wheel.

File: legged_examples/legged_unitree/legged_unitree_description/urdf/common/leg.xacro (robot description, xacro)
@@ -2,5 +2,5 @@
 <robot xmlns:xacro="http://www.ros.org/wiki/xacro">
     <xacro:include filename="$(find legged_unitree_description)/urdf/common/transmission.xacro"/>
-    <xacro:macro name="leg" params="prefix mesh_path mirror mirror_dae front_hind front_hind_dae *origin">
+    <xacro:macro name="leg" params="prefix mesh_path mirror mirror_dae wheel front_hind front_hind_dae *origin">
         <joint name="${prefix}_HAA" type="revolute">
             <xacro:insert_block name="origin"/>
@@ -104,5 +104,6 @@
             <axis xyz="0 1 0"/>
             <dynamics damping="${damping}" friction="${friction}"/>
-            <limit effort="${calf_torque_max}" velocity="${calf_velocity_max}" lower="${calf_position_min}" upper="${calf_position_max}"/>
+            <limit effort="${calf_torque_max}" velocity="${calf_velocity_max}" lower="${calf_position_min}"
+                   upper="${calf_position_max}"/>
         </joint>
         <link name="${prefix}_calf">
@@ -110,6 +111,10 @@
                 <origin rpy="0 0 0" xyz="0 0 0"/>
                 <geometry>
-                    <mesh filename="${mesh_path}/calf.dae"
-                          scale="1 1 1"/>
+                    <xacro:if value="${(mirror_dae == False) and (wheel == True)}">
+                        <mesh filename="${mesh_path}/calf_mirror.dae" scale="1 1 1"/>
+                    </xacro:if>
+                    <xacro:unless value="${(mirror_dae == False) and (wheel == True)}">
+                        <mesh filename="${mesh_path}/calf.dae" scale="1 1 1"/>
+                    </xacro:unless>
                 </geometry>
                 <material name="orange"/>
@@ -130,34 +135,80 @@
             </inertial>
         </link>
-        <joint name="${prefix}_foot_fixed" type="fixed" dont_collapse="true">
-            <origin rpy="0 0 0" xyz="0 0 ${-(calf_length)}"/>
-            <parent link="${prefix}_calf"/>
-            <child link="${prefix}_FOOT"/>
-        </joint>
-        <link name="${prefix}_FOOT">
-            <visual>
-                <origin rpy="0 0 0" xyz="0 0 0"/>
-                <geometry>
-                    <sphere radius="${foot_radius-0.01}"/>
-                </geometry>
-                <material name="orange"/>
-            </visual>
-            <collision>
-                <origin rpy="0 0 0" xyz="0 0 0"/>
-                <geometry>
-                    <sphere radius="${foot_radius}"/>
-                </geometry>
-            </collision>
-            <inertial>
-                <mass value="${foot_mass}"/>
-                <inertia
-                        ixx="${(2*foot_mass)/5.0*(foot_radius*foot_radius)}" ixy="0.0" ixz="0.0"
-                        iyy="${(2*foot_mass)/5.0*(foot_radius*foot_radius)}" iyz="0.0"
-                        izz="${(2*foot_mass)/5.0*(foot_radius*foot_radius)}"/>
-            </inertial>
-        </link>
-        <gazebo reference="${prefix}_foot_fixed">
-            <disableFixedJointLumping>true</disableFixedJointLumping>
-        </gazebo>
+        <xacro:if value="${(wheel == True)}">
+            <joint name="${prefix}_foot_joint" type="continuous">
+                <xacro:if value="${mirror_dae == True}">
+                    <origin rpy="0 0 0" xyz="0 0 ${-(calf_length)}"/>
+                </xacro:if>
+                <xacro:if value="${mirror_dae == False}">
+                    <origin rpy="0 0 0" xyz="0 -0.001 ${-(calf_length)}"/>
+                </xacro:if>
+                <parent link="${prefix}_calf"/>
+                <child link="${prefix}_FOOT"/>
+                <axis xyz="0 1 0"/>
+                <limit effort="20" velocity="50"/>
+            </joint>
+            <link name="${prefix}_FOOT">
+                <inertial>
+                    <origin xyz="-0.000991 -0.051053 -0.00113" rpy="0 0 0"/>
+                    <mass value="1.083"/>
+                    <inertia ixx="0.004121" ixy="-6E-06" ixz="-4.8E-05" iyy="0.007776" iyz="-7E-06" izz="0.004108"/>
+                </inertial>
+                <visual>
+                    <origin xyz="0 0 0" rpy="0 0 0"/>
+                    <geometry>
+                        <mesh filename="${mesh_path}/${prefix}_foot.dae"/>
+                    </geometry>
+                    <material name="黑色硅胶-effect">
+                        <color rgba="0.073 0.073 0.073 1"/>
+                    </material>
+                </visual>
+                <collision>
+                    <origin xyz="0 0 0" rpy="0 0 0"/>
+                    <geometry>
+                        <mesh filename="${mesh_path}/${prefix}_foot.dae"/>
+                    </geometry>
+                </collision>
+            </link>
+        </xacro:if>
+        <xacro:if value="${(wheel == False)}">
+            <joint name="${prefix}_foot_fixed" type="fixed" dont_collapse="true">
+                <origin rpy="0 0 0" xyz="0 0 ${-(calf_length)}"/>
+                <parent link="${prefix}_calf"/>
+                <child link="${prefix}_FOOT"/>
+            </joint>
+            <link name="${prefix}_FOOT">
+                <visual>
+                    <origin rpy="0 0 0" xyz="0 0 0"/>
+                    <geometry>
+                        <sphere radius="${foot_radius-0.01}"/>
+                    </geometry>
+                    <material name="orange"/>
+                </visual>
+                <collision>
+                    <origin rpy="0 0 0" xyz="0 0 0"/>
+                    <geometry>
+                        <sphere radius="${foot_radius}"/>
+                    </geometry>
+                </collision>
+                <inertial>
+                    <mass value="${foot_mass}"/>
+                    <inertia
+                            ixx="${(2*foot_mass)/5.0*(foot_radius*foot_radius)}" ixy="0.0" ixz="0.0"
+                            iyy="${(2*foot_mass)/5.0*(foot_radius*foot_radius)}" iyz="0.0"
+                            izz="${(2*foot_mass)/5.0*(foot_radius*foot_radius)}"/>
+                </inertial>
+            </link>
+            <gazebo reference="${prefix}_foot_fixed">
+                <disableFixedJointLumping>true</disableFixedJointLumping>
+            </gazebo>
+            <gazebo reference="${prefix}_FOOT">
+                <mu1>0.6</mu1>
+                <mu2>0.6</mu2>
+                <self_collide>1</self_collide>
+                <material>Gazebo/DarkGrey</material>
+                <kp value="1000000.0"/>
+                <kd value="100.0"/>
+            </gazebo>
+        </xacro:if>
         <gazebo reference="${prefix}_hip">
             <mu1>0.2</mu1>
@@ -178,12 +229,4 @@
             <self_collide>1</self_collide>
         </gazebo>
-        <gazebo reference="${prefix}_FOOT">
-            <mu1>0.6</mu1>
-            <mu2>0.6</mu2>
-            <self_collide>1</self_collide>
-            <material>Gazebo/DarkGrey</material>
-            <kp value="1000000.0"/>
-            <kd value="100.0"/>
-        </gazebo>
         <xacro:leg_transmission name="${prefix}"/>
     </xacro:macro>

File: legged_examples/legged_unitree/legged_unitree_description/urdf/robot.xacro (robot description, xacro)
@@ -7,5 +7,5 @@
     <xacro:include filename="$(find legged_unitree_description)/urdf/common/imu.xacro"/>
     <xacro:include filename="$(find legged_unitree_description)/urdf/$(arg robot_type)/const.xacro"/>
-<!--    <xacro:property name="mesh_path" value="../meshes"/>-->
+    <!--    <xacro:property name="mesh_path" value="../meshes"/>-->
     <xacro:property name="mesh_path" value="package://legged_unitree_description/meshes/$(arg robot_type)"/>
     <link name="base">
@@ -32,14 +32,18 @@
     </link>
     <xacro:IMU connected_to="base" imu_name="base_imu" xyz="0. 0. 0." rpy="0. 0. 0."/>
-    <xacro:leg prefix="LF" mesh_path="${mesh_path}" mirror="1" mirror_dae="True" front_hind="1" front_hind_dae="True">
+    <xacro:leg prefix="LF" mesh_path="${mesh_path}" mirror="1" mirror_dae="True" wheel="True" front_hind="1"
+               front_hind_dae="True">
         <origin rpy="0 0 0" xyz="${leg_offset_x} ${leg_offset_y} 0"/>
     </xacro:leg>
-    <xacro:leg prefix="LH" mesh_path="${mesh_path}" mirror="1" mirror_dae="True" front_hind="-1" front_hind_dae="False">
+    <xacro:leg prefix="LH" mesh_path="${mesh_path}" mirror="1" mirror_dae="True" wheel="True" front_hind="-1"
+               front_hind_dae="False">
         <origin rpy="0 0 0" xyz="${-leg_offset_x} ${leg_offset_y} 0"/>
     </xacro:leg>
-    <xacro:leg prefix="RF" mesh_path="${mesh_path}" mirror="-1" mirror_dae="False" front_hind="1" front_hind_dae="True">
+    <xacro:leg prefix="RF" mesh_path="${mesh_path}" mirror="-1" mirror_dae="False" wheel="True" front_hind="1"
+               front_hind_dae="True">
         <origin rpy="0 0 0" xyz="${leg_offset_x} ${-leg_offset_y} 0"/>
     </xacro:leg>
-    <xacro:leg prefix="RH" mesh_path="${mesh_path}" mirror="-1" mirror_dae="False" front_hind="-1" front_hind_dae="False">
+    <xacro:leg prefix="RH" mesh_path="${mesh_path}" mirror="-1" mirror_dae="False" wheel="True" front_hind="-1"
+               front_hind_dae="False">
         <origin rpy="0 0 0" xyz="${-leg_offset_x} ${-leg_offset_y} 0"/>
     </xacro:leg>

Commit message: Modify dir name.

File: legged_examples/legged_unitree/legged_unitree_description/urdf/common/leg.xacro (robot description, xacro)
@@ -136,5 +136,5 @@
         </link>
         <xacro:if value="${(wheel == True)}">
-            <joint name="${prefix}_foot_joint" type="continuous">
+            <joint name="${prefix}_foot_joint" type="fixed">
                 <xacro:if value="${mirror_dae == True}">
                     <origin rpy="0 0 0" xyz="0 0 ${-(calf_length)}"/>
@@ -229,5 +229,5 @@
             <self_collide>1</self_collide>
         </gazebo>
-        <xacro:leg_transmission name="${prefix}"/>
+        <xacro:leg_transmission name="${prefix}" wheel="${wheel}"/>
     </xacro:macro>
 </robot>

File: legged_examples/legged_unitree/legged_unitree_description/urdf/common/transmission.xacro (robot description, xacro)
@@ -1,5 +1,5 @@
 <?xml version="1.0"?>
 <robot xmlns:xacro="http://www.ros.org/wiki/xacro">
-    <xacro:macro name="leg_transmission" params="name">
+    <xacro:macro name="leg_transmission" params="name wheel">
         <transmission name="${prefix}_HAA_tran">
             <type>transmission_interface/SimpleTransmission</type>
@@ -32,4 +32,16 @@
             </actuator>
         </transmission>
+        <!--        <xacro:if value="${wheel==True}">-->
+        <!--            <transmission name="${prefix}_foot_tran">-->
+        <!--                <type>transmission_interface/SimpleTransmission</type>-->
+        <!--                <joint name="${prefix}_foot_joint">-->
+        <!--                    <hardwareInterface>hardware_interface/EffortJointInterface</hardwareInterface>-->
+        <!--                </joint>-->
+        <!--                <actuator name="${prefix}_foot_motor">-->
+        <!--                    <hardwareInterface>hardware_interface/EffortJointInterface</hardwareInterface>-->
+        <!--                    <mechanicalReduction>1</mechanicalReduction>-->
+        <!--                </actuator>-->
+        <!--            </transmission>-->
+        <!--        </xacro:if>-->
     </xacro:macro>
 </robot>
