Commit message: Add b2w urdf and add standup mode.

File: legged_examples/legged_unitree/legged_unitree_description/urdf/a1/const.xacro (robot description, xacro)
@@ -90,3 +90,4 @@
     <!-- foot -->
     <xacro:property name="foot_mass" value="0.06"/>
+    <xacro:property name="wheel" value="False"/>
 </robot>

File: legged_examples/legged_unitree/legged_unitree_description/urdf/b2w/const.xacro (robot description, xacro)
@@ -121,3 +121,4 @@
     <!-- foot -->
     <xacro:property name="foot_mass" value="0.098183"/>
+    <xacro:property name="wheel" value="True"/>
 </robot>

File: legged_examples/legged_unitree/legged_unitree_description/urdf/common/leg.xacro (robot description, xacro)
@@ -136,5 +136,5 @@
         </link>
         <xacro:if value="${(wheel == True)}">
-            <joint name="${prefix}_foot_joint" type="fixed">
+            <joint name="${prefix}_foot_joint" type="revolute">
                 <xacro:if value="${mirror_dae == True}">
                     <origin rpy="0 0 0" xyz="0 0 ${-(calf_length)}"/>
@@ -164,7 +164,12 @@
                 </visual>
                 <collision>
-                    <origin xyz="0 0 0" rpy="0 0 0"/>
-                    <geometry>
-                        <mesh filename="${mesh_path}/${prefix}_foot.dae"/>
+                    <xacro:if value="${mirror_dae == True}">
+                        <origin rpy="${pi/2} 0 0" xyz="0 0.045 0"/>
+                    </xacro:if>
+                    <xacro:if value="${mirror_dae == False}">
+                        <origin rpy="${pi/2} 0 0" xyz="0 -0.045 0"/>
+                    </xacro:if>
+                    <geometry>
+                        <cylinder length="0.02" radius="0.1125"/>
                     </geometry>
                 </collision>
@@ -202,12 +207,4 @@
                 <disableFixedJointLumping>true</disableFixedJointLumping>
             </gazebo>
-            <gazebo reference="${prefix}_FOOT">
-                <mu1>0.6</mu1>
-                <mu2>0.6</mu2>
-                <self_collide>1</self_collide>
-                <material>Gazebo/DarkGrey</material>
-                <kp value="1000000.0"/>
-                <kd value="100.0"/>
-            </gazebo>
         </xacro:if>
         <gazebo reference="${prefix}_hip">
@@ -229,4 +226,12 @@
             <self_collide>1</self_collide>
         </gazebo>
+        <gazebo reference="${prefix}_FOOT">
+            <mu1>0.6</mu1>
+            <mu2>0.6</mu2>
+            <self_collide>1</self_collide>
+            <material>Gazebo/DarkGrey</material>
+            <kp value="1000000.0"/>
+            <kd value="100.0"/>
+        </gazebo>
         <xacro:leg_transmission name="${prefix}" wheel="${wheel}"/>
     </xacro:macro>

File: legged_examples/legged_unitree/legged_unitree_description/urdf/common/transmission.xacro (robot description, xacro)
@@ -32,16 +32,16 @@
             </actuator>
         </transmission>
-        <!--        <xacro:if value="${wheel==True}">-->
-        <!--            <transmission name="${prefix}_foot_tran">-->
-        <!--                <type>transmission_interface/SimpleTransmission</type>-->
-        <!--                <joint name="${prefix}_foot_joint">-->
-        <!--                    <hardwareInterface>hardware_interface/EffortJointInterface</hardwareInterface>-->
-        <!--                </joint>-->
-        <!--                <actuator name="${prefix}_foot_motor">-->
-        <!--                    <hardwareInterface>hardware_interface/EffortJointInterface</hardwareInterface>-->
-        <!--                    <mechanicalReduction>1</mechanicalReduction>-->
-        <!--                </actuator>-->
-        <!--            </transmission>-->
-        <!--        </xacro:if>-->
+        <xacro:if value="${wheel==True}">
+            <transmission name="${prefix}_foot_tran">
+                <type>transmission_interface/SimpleTransmission</type>
+                <joint name="${prefix}_foot_joint">
+                    <hardwareInterface>hardware_interface/EffortJointInterface</hardwareInterface>
+                </joint>
+                <actuator name="${prefix}_foot_motor">
+                    <hardwareInterface>hardware_interface/EffortJointInterface</hardwareInterface>
+                    <mechanicalReduction>1</mechanicalReduction>
+                </actuator>
+            </transmission>
+        </xacro:if>
     </xacro:macro>
 </robot>

File: legged_examples/legged_unitree/legged_unitree_description/urdf/robot.xacro (robot description, xacro)
@@ -32,17 +32,17 @@
     </link>
     <xacro:IMU connected_to="base" imu_name="base_imu" xyz="0. 0. 0." rpy="0. 0. 0."/>
-    <xacro:leg prefix="LF" mesh_path="${mesh_path}" mirror="1" mirror_dae="True" wheel="True" front_hind="1"
+    <xacro:leg prefix="LF" mesh_path="${mesh_path}" mirror="1" mirror_dae="True" wheel="${wheel}" front_hind="1"
                front_hind_dae="True">
         <origin rpy="0 0 0" xyz="${leg_offset_x} ${leg_offset_y} 0"/>
     </xacro:leg>
-    <xacro:leg prefix="LH" mesh_path="${mesh_path}" mirror="1" mirror_dae="True" wheel="True" front_hind="-1"
+    <xacro:leg prefix="LH" mesh_path="${mesh_path}" mirror="1" mirror_dae="True" wheel="${wheel}" front_hind="-1"
                front_hind_dae="False">
         <origin rpy="0 0 0" xyz="${-leg_offset_x} ${leg_offset_y} 0"/>
     </xacro:leg>
-    <xacro:leg prefix="RF" mesh_path="${mesh_path}" mirror="-1" mirror_dae="False" wheel="True" front_hind="1"
+    <xacro:leg prefix="RF" mesh_path="${mesh_path}" mirror="-1" mirror_dae="False" wheel="${wheel}" front_hind="1"
                front_hind_dae="True">
         <origin rpy="0 0 0" xyz="${leg_offset_x} ${-leg_offset_y} 0"/>
     </xacro:leg>
-    <xacro:leg prefix="RH" mesh_path="${mesh_path}" mirror="-1" mirror_dae="False" wheel="True" front_hind="-1"
+    <xacro:leg prefix="RH" mesh_path="${mesh_path}" mirror="-1" mirror_dae="False" wheel="${wheel}" front_hind="-1"
                front_hind_dae="False">
         <origin rpy="0 0 0" xyz="${-leg_offset_x} ${-leg_offset_y} 0"/>
